File: DX32D.kicad_sch (KiCad schematic)
At the start: 20 parts, among them J1 USB_A, J2 MicroSD Card, J3 SH I2C, SW1 reset, SW2 boot, U1 ESP32-S3-WROOM-1, U2 AMS1117-3.3

Commit message: made some small changes
Connections:
- no-connect marks 31 -> 30
Changed lines of the file:
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@@
-	)
-	(no_connect
-		(at 137.16 140.97)
 	)
 	(no_connect
